File: pcb/wristpad.kicad_pcb (KiCad board)
At the start: 4 copper layers, 40 x 38.3 mm, 74 parts, among them IC1 AS5600-ASOT, J1 USB4105-GF-A, J2 Conn_01x02, Q1 DMN2004VK-7, Q2 DMP2004VK-7, Q3 DMN2004VK-7, SW1 EN, SW2 BOOT, SW3 B1, SW4 B2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

Commit message: panelized, fixes
Parts:
- L1: value TBD -> 0R
- SW1: value EN -> top-switch
- SW2: value BOOT -> top-switch
- SW3: value B1 -> side-switch
- SW4: value B2 -> side-switch
- SW5: value B3 -> side-switch
Routing:
- net VBUS: track 72.1 -> 73.9 mm
Other:
- board text removed: "JLCJLCJLCJLC"
