File: pcb/disqo.kicad_pcb (KiCad board)
At the start: 4 copper layers, 40 x 38.3 mm, 74 parts, among them IC1 AS5600-ASOT, J1 USB4105-GF-A, J2 Conn_01x02, Q1 DMN2004VK-7, Q2 DMP2004VK-7, Q3 DMN2004VK-7, SW1 top-switch, SW2 top-switch, SW3 side-switch, SW4 side-switch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

Commit message: rename
Routing:
- net /PIEZO_GATE: track 6.14 -> 5.60 mm
