File: pcb/disqo.kicad_pcb (KiCad board)
At the start: 4 copper layers, 40 x 37 mm, 74 parts, among them IC1 AS5600-ASOT, J1 USB4105-GF-A, J2 Conn_01x02, Q1 DMN2004VK-7, Q2 DMP2004VK-7, Q3 DMN2004VK-7, SW1 top-switch, SW3 side-switch, SW4 side-switch, SW5 side-switch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

Commit message: pcb changes
Parts:
- R16, R20, R3, R32, R33, R34: value 100k -> 1M
Routing:
- net /CONNECTED: track 23.9 -> 25.1 mm
Other:
- board text added: "TODO: remove the pull-up/down resistor on the piezo gate TODO: make sure the connected pin's pull resistors are actually connected TODO: just remove the reset button TODO: can we somehow benefit from a passive low pass filter on the piezo?"
- board text removed: "TODO: exposed gnd and other areas for crocodile clips in the unused space"
Changed lines of the file:
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@@
       (effects (font (size 0.8 0.8) (thickness 0.15)))
     )
-    (fp_text value "100k" (at 0 1.17) (layer "F.Fab")
+    (fp_text value "1M" (at 0 1.17) (layer "F.Fab")
       (effects (font (size 1 1) (thickness 0.15)))
     )
@@
       (effects (font (size 0.8 0.8) (thickness 0.15)))
     )
-    (fp_text value "100k" (at 0 1.17 90) (layer "F.Fab")
+    (fp_text value "1M" (at 0 1.17 90) (layer "F.Fab")
       (effects (font (size 1 1) (thickness 0.15)))
     )
@@
       (effects (font (size 1 1) (thickness 0.15)))
     )
-    (fp_text value "100k" (at 0 1.17) (layer "F.Fab")
+    (fp_text value "1M" (at 0 1.17) (layer "F.Fab")
       (effects (font (size 1 1) (thickness 0.15)))
     )
@@
       (effects (font (size 0.8 0.8) (thickness 0.15)))
     )
-    (fp_text value "100k" (at 0 1.17) (layer "F.Fab")
+    (fp_text value "1M" (at 0 1.17) (layer "F.Fab")
       (effects (font (size 1 1) (thickness 0.15)))
     )
@@
       (effects (font (size 1 1) (thickness 0.15)))
     )
-    (fp_text value "100k" (at 0 1.17) (layer "F.Fab")
+    (fp_text value "1M" (at 0 1.17) (layer "F.Fab")
       (effects (font (size 1 1) (thickness 0.15)))
     )
@@
       (effects (font (size 1 1) (thickness 0.15)))
     )
-    (fp_text value "100k" (at 0 1.17) (layer "F.Fab")
+    (fp_text value "1M" (at 0 1.17) (layer "F.Fab")
       (effects (font (size 1 1) (thickness 0.15)))
     )
@@
   (gr_line (start 92.77 84) (end 92.77 116) (layer "User.3") (width 0.15))
   (gr_line (start 112.77 84) (end 112.77 116) (layer "User.3") (width 0.15))
-  (gr_text "TODO: exposed gnd and other areas for crocodile clips in the unused space" (at 97 132) (layer "User.1")
+  (gr_text "TODO: remove the pull-up/down resistor on the piezo gate\nTODO: make sure the connected pin's pull resistors are actually connected\nTODO: just remove the reset button\nTODO: can we somehow benefit from a passive low pass filter on the piezo?" (at 97 132) (layer "User.1")
     (effects (font (size 1.5 1.5) (thickness 0.3)))
   )
@@
   (segment (start 99.45 98.79) (end 99.45 99.33) (width 0.2) (layer "B.Cu") (net 7))
   (segment (start 97.351014 96.691014) (end 99.45 98.79) (width 0.2) (layer "B.Cu") (net 7))
+  (segment (start 105.25 99.645082) (end 105.25 97.95) (width 0.2) (layer "F.Cu") (net 8))
   (segment (start 112.6 107) (end 112.63 107.03) (width 0.2) (layer "F.Cu") (net 8))
   (segment (start 112 107) (end 112.6 107) (width 0.2) (layer "F.Cu") (net 8))
-  (segment (start 105.25 99.645082) (end 105.25 97.95) (width 0.2) (layer "F.Cu") (net 8))
   (segment (start 106.801604 101.196686) (end 105.25 99.645082) (width 0.2) (layer "F.Cu") (net 8))
   (via (at 106.801604 101.196686) (size 0.6) (drill 0.3) (layers "F.Cu" "B.Cu") (net 8))
@@
   (segment (start 108.5 106) (end 108.55 105.95) (width 0.2) (layer "F.Cu") (net 52))
   (segment (start 108.32 94.95) (end 107.65 94.95) (width 0.2) (layer "F.Cu") (net 52))
+  (segment (start 107.51 105.5) (end 108 105.5) (width 0.2) (layer "F.Cu") (net 52))
   (segment (start 108.55 101.210051) (end 109.2 100.560052) (width 0.2) (layer "F.Cu") (net 52))
   (segment (start 107.5625 112.5) (end 106.9 112.5) (width 0.2) (layer "F.Cu") (net 52))
@@
   (segment (start 109.2 95.83) (end 108.32 94.95) (width 0.2) (layer "F.Cu") (net 52))
   (segment (start 108.55 105.95) (end 108.55 101.210051) (width 0.2) (layer "F.Cu") (net 52))
+  (segment (start 108 105.5) (end 108.5 106) (width 0.2) (layer "F.Cu") (net 52))
   (segment (start 107.51 104.5) (end 107.51 105.5) (width 0.2) (layer "F.Cu") (net 52))
   (segment (start 106.9 112.5) (end 106.41 112.99) (width 0.2) (layer "F.Cu") (net 52))
@@
   (segment (start 104.35 95.75) (end 107.65 95.75) (width 0.2) (layer "F.Cu") (net 57))
   (via (at 104.32 95.72) (size 0.6) (drill 0.3) (layers "F.Cu" "B.Cu") (net 57))
-  (segment (start 104.142182 95.72) (end 101.06 98.802182) (width 0.2) (layer "B.Cu") (net 57))
-  (segment (start 101.05 100.847818) (end 101.05 108.5195) (width 0.2) (layer "B.Cu") (net 57))
   (segment (start 100.7 108.8695) (end 100.7 110.0195) (width 0.2) (layer "B.Cu") (net 57))
-  (segment (start 100.71 99.607818) (end 101.032182 99.93) (width 0.2) (layer "B.Cu") (net 57))
-  (segment (start 104.32 95.72) (end 104.142182 95.72) (width 0.2) (layer "B.Cu") (net 57))
+  (segment (start 101.05 100.847818) (end 101.05 108.5195) (width 0.2) (layer "B.Cu") (net 57))
+  (segment (start 104.142182 95.72) (end 100.7 99.162182) (width 0.2) (layer "B.Cu") (net 57))
   (segment (start 101.05 108.5195) (end 100.7 108.8695) (width 0.2) (layer "B.Cu") (net 57))
-  (segment (start 101.06 98.802182) (end 101.06 98.83) (width 0.2) (layer "B.Cu") (net 57))
-  (segment (start 101.032182 99.93) (end 101.06 99.93) (width 0.2) (layer "B.Cu") (net 57))
-  (segment (start 100.86 100.202182) (end 100.86 100.657818) (width 0.2) (layer "B.Cu") (net 57))
-  (segment (start 101.06 98.83) (end 101.032182 98.83) (width 0.2) (layer "B.Cu") (net 57))
-  (segment (start 101.06 99.93) (end 101.06 100.002182) (width 0.2) (layer "B.Cu") (net 57))
-  (segment (start 100.86 100.657818) (end 101.05 100.847818) (width 0.2) (layer "B.Cu") (net 57))
-  (segment (start 101.06 100.002182) (end 100.86 100.202182) (width 0.2) (layer "B.Cu") (net 57))
-  (segment (start 100.71 99.152182) (end 100.71 99.607818) (width 0.2) (layer "B.Cu") (net 57))
-  (segment (start 101.032182 98.83) (end 100.71 99.152182) (width 0.2) (layer "B.Cu") (net 57))
+  (segment (start 100.7 99.162182) (end 100.7 100.497818) (width 0.2) (layer "B.Cu") (net 57))
+  (segment (start 104.32 95.72) (end 104.142182 95.72) (width 0.2) (layer "B.Cu") (net 57))
+  (segment (start 100.7 100.497818) (end 101.05 100.847818) (width 0.2) (layer "B.Cu") (net 57))
   (segment (start 108.25 111.3125) (end 108.25 110.23) (width 0.4) (layer "F.Cu") (net 58))
   (segment (start 108.75 110.27) (end 108.48 110) (width 0.4) (layer "F.Cu") (net 58))

Commit message: wip
Parts:
- R16, R20: value 1M -> 10k
- R3, R32, R33, R34: value 1M -> 100k
Changed lines of the file:
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@@
       (effects (font (size 0.8 0.8) (thickness 0.15)))
     )
-    (fp_text value "1M" (at 0 1.17) (layer "F.Fab")
+    (fp_text value "10k" (at 0 1.17) (layer "F.Fab")
       (effects (font (size 1 1) (thickness 0.15)))
     )
@@
       (effects (font (size 0.8 0.8) (thickness 0.15)))
     )
-    (fp_text value "1M" (at 0 1.17 90) (layer "F.Fab")
+    (fp_text value "100k" (at 0 1.17 90) (layer "F.Fab")
       (effects (font (size 1 1) (thickness 0.15)))
     )
@@
       (effects (font (size 1 1) (thickness 0.15)))
     )
-    (fp_text value "1M" (at 0 1.17) (layer "F.Fab")
+    (fp_text value "100k" (at 0 1.17) (layer "F.Fab")
       (effects (font (size 1 1) (thickness 0.15)))
     )
@@
       (effects (font (size 0.8 0.8) (thickness 0.15)))
     )
-    (fp_text value "1M" (at 0 1.17) (layer "F.Fab")
+    (fp_text value "10k" (at 0 1.17) (layer "F.Fab")
       (effects (font (size 1 1) (thickness 0.15)))
     )
@@
       (effects (font (size 1 1) (thickness 0.15)))
     )
-    (fp_text value "1M" (at 0 1.17) (layer "F.Fab")
+    (fp_text value "100k" (at 0 1.17) (layer "F.Fab")
       (effects (font (size 1 1) (thickness 0.15)))
     )
@@
       (effects (font (size 1 1) (thickness 0.15)))
     )
-    (fp_text value "1M" (at 0 1.17) (layer "F.Fab")
-      (effects (font (size 1 1) (thickness 0.15)))
-    )
+    (fp_text value "100k" (at 0 1.17) (layer "F.Fab")
+      (effects (font (size 1 1) (thickness 0.15)))
+    )
