File: pcb/disqo.kicad_sch (KiCad schematic)
At the start: 75 parts, among them IC1 AS5600-ASOT, J1 USB4105-GF-A, J2 Conn_01x02, Q1 DMN2004VK-7, Q2 DMP2004VK-7, Q3 DMN2004VK-7, SW1 top-switch, SW2 top-switch, SW3 side-switch, SW4 side-switch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

Commit message: rename
Parts:
- C18, C19: now left out of the parts list
Changed lines of the file:
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@@
   )
   (symbol (lib_id "Device:C_Small") (at 184.15 64.135 0) (unit 1)
-    (in_bom yes) (on_board yes) (fields_autoplaced)
+    (in_bom no) (on_board yes) (fields_autoplaced)
     (property "Reference" "C18" (id 0) (at 186.4741 63.3066 0)
       (effects (font (size 1.27 1.27)) (justify left))
@@
   )
   (symbol (lib_id "Device:C_Small") (at 196.215 64.135 0) (unit 1)
-    (in_bom yes) (on_board yes) (fields_autoplaced)
+    (in_bom no) (on_board yes) (fields_autoplaced)
     (property "Reference" "C19" (id 0) (at 198.5391 63.3066 0)
       (effects (font (size 1.27 1.27)) (justify left))

Commit message: PCB tweaks
Parts:
- removed TP3: RTS, TestPoint:TestPoint_Pad_D1.0mm, symbol Connector:TestPoint_Small
- removed TP4: DTR, TestPoint:TestPoint_Pad_D1.0mm, symbol Connector:TestPoint_Small
- added R28: 0R, Resistor_SMD:R_0805_2012Metric, symbol Device:R_Small
- added R29, R30, R31: 10k, Resistor_SMD:R_0402_1005Metric, symbol Device:R_Small
- C1, C16, C4, C5, C8: footprint Capacitor_SMD:C_0402_1005Metric -> Capacitor_SMD:C_0805_2012Metric
- L1: footprint Inductor_SMD:L_0603_1608Metric -> Inductor_SMD:L_0805_2012Metric
- R13: value 10k -> 1k
- R18, R19: value 4.7k -> 5.1k
- TP1, TP2, TP6, TP7: footprint TestPoint:TestPoint_Pad_D1.0mm -> testpoint:TestPoint_Pad_D1.0mm
Connections:
- net +3V3: now also R29.2, R30.2, R31.2; no longer R18.1, R19.2
- net B1: now also SW3.1, R29.1; no longer SW3.2
- net B2: now also SW4.1, R30.1; no longer SW4.2
- net B3: now also R31.1
- net CONNECTED: now also U3.32 (SD_DATA_0/GPIO7); no longer U3.16 (GPIO27/ADC2_CH7/RTC_GPIO17)
- net ENABLE: now also U3.16 (GPIO27/ADC2_CH7/RTC_GPIO17); no longer U3.33 (SD_DATA_1/GPIO8)
- net GND: now also SW3.2, SW4.2; no longer SW3.1, SW4.1
- net PIEZO: now also U3.34 (*GPIO5); no longer U3.27 (GPIO20)
- net POWER: now also R18.1, R19.2
- net SCL: no longer U5.9 (SCL)
- net SDA: no longer U5.10 (SDA)
- net VCC: now also R28.2; no longer D2.1 (K), Q2.1 (S)
- net SCLK: now reaches U3.17 (MTMS/GPIO14/ADC2_CH6/RTC_GPIO16)
- net SCLK: now also U5.9 (SCL)
- net MOSI: now reaches U3.20 (MTCK/GPIO13/ADC2_CH4/RTC_GPIO14)
- net MOSI: now also U5.10 (SDA)
- net CS: now reaches U3.21 (*MTDO/GPIO15/ADC2_CH3/RTC_GPIO13)
- net CS: now also U5.8 (CS)
- net LCD_RESET: now reaches U5.11 (RESET)
- net LCD_RESET: now also U3.33 (SD_DATA_1/GPIO8)
- net LCD_DC: now reaches U5.7 (D/C)
- net LCD_DC: now also U3.27 (GPIO20)
- net VO renamed VOUT
- new net VOR: D2.1 (K), Q2.1 (S), R28.1
- no-connect marks 25 -> 17
Other:
- note added: "10k, 1uf ideally"
- note added: "GPIO37, GPIO38, GPIO39 do not have pull-ups."
- note added: "TODO: BOOT seems to be low on power-up :( probably without cp2102n"
- note added: "TODO: test points for voltages, both sides of each diode"
- note added: "finicky as hell"
- note removed: "FREE"
- note removed: "TODO: should we rather go with discrete rather than dual packages?"
- moved on the sheet: C10, Q3A, R15, R17, R18, R19, R20, SW3, SW4, SW5, U5

Commit message: pcb changes
Parts:
- removed C12: 0.1uF, Capacitor_SMD:C_0402_1005Metric, symbol Device:C_Small
- removed C18, C19: TBD, Capacitor_SMD:C_0603_1608Metric, symbol Device:C_Small
- removed E1: 2450AT42E0100E, 2450AT42E0100:XDCR_2450AT42E0100E, symbol 2450AT42E0100E:2450AT42E0100E
- removed L1: 0R, Inductor_SMD:L_0805_2012Metric, symbol Device:L_Small
- removed SW2: top-switch, KXT-311:KXT 311 LHS, symbol Switch:SW_Push
- removed TP6: TXD, testpoint:TestPoint_Pad_D1.0mm, symbol Connector:TestPoint_Small
- removed TP7: RXD, testpoint:TestPoint_Pad_D1.0mm, symbol Connector:TestPoint_Small
- removed U3: ESP32-PICO-V3, Package_DFN_QFN:QFN-48-1EP_7x7mm_P0.5mm_EP5.15x5.15mm, symbol Espressif:ESP32-PICO-V3
- added R32, R33, R34: 100k, Resistor_SMD:R_0402_1005Metric, symbol Device:R_Small
- added TP3, TP4: GND, tab:tab, symbol Connector:TestPoint_Small
- added U3: ESP32-PICO-MINI-02, Espressif:ESP32-PICO-MINI-02_Hand-Soldering, symbol Espressif:ESP32-PICO-MINI-02
- C15: value 0.1uF -> 1uF; footprint Capacitor_SMD:C_0402_1005Metric -> Capacitor_SMD:C_0603_1608Metric
- C16: value 10uF -> 22uF
- J2: footprint battery-connector:Battery Connector -> Connector_JST:JST_ACH_BM02B-ACHSS-GAN-ETF_1x02-1MP_P1.20mm_Vertical
- R13: value 1k -> 10k
- R14: footprint (none) -> Resistor_SMD:R_0603_1608Metric
- TP1: value DAC1 -> BATT+; footprint testpoint:TestPoint_Pad_D1.0mm -> TestPoint:TestPoint_THTPad_D1.5mm_Drill0.7mm
- TP2: value DAC2 -> GND; footprint testpoint:TestPoint_Pad_D1.0mm -> TestPoint:TestPoint_THTPad_D1.5mm_Drill0.7mm
Connections:
- net +3V3: now also U3.3 (3V3)
- net +BATT: now also TP1.1
- net 32K_XN: now also U3.13 (32K_XN/GPIO33/ADC1_CH5)
- net 32K_XP: now also U3.12 (32K_XP/GPIO32/ADC1_CH4)
- net B1: now also U3.5 (SENSOR_CAPP/GPIO37/ADC1_CH1)
- net B2: now also U3.6 (SENSOR_CAPN/GPIO38/ADC1_CH2)
- net B3: now also U3.7 (SENSOR_VN/GPIO39/ADC1_CH3)
- net BACKLIGHT: now also U3.33 (GPIO19)
- net BATT_ADC: now also U3.9 (VDET_1/GPIO34/ADC1_CH6)
- net BOOT: now also U3.23 (*GPIO0/BOOT/ADC2_CH1)
- net CONNECTED: now also U3.27 (SD_DATA_0/GPIO7)
- net CS: now also U3.21 (*MTDO/GPIO15/ADC2_CH3)
- net DAC1: now also U3.15 (GPIO25/ADC2_CH8/DAC_1); no longer TP1.1
- net DAC2: now also U3.16 (GPIO26/ADC2_CH9/DAC_2); no longer TP2.1
- net DTR_BASE: now also R32.1
- net EN: now also U3.8 (EN/CHIP_PU)
- net ENABLE: now also U3.17 (GPIO27/ADC2_CH7)
- net GND: now also TP2.1, R32.2, R33.2, R34.2, TP3.1, TP4.1, U3.1 (GND), U3.11 (GND), U3.14 (GND), U3.2 (GND), U3.36 (GND)
- net LCD_DC: now also U3.26 (GPIO20)
- net LCD_RESET: now also U3.28 (SD_DATA_1/GPIO8)
- net MOSI: now also U3.20 (MTCK/GPIO13/ADC2_CH4)
- net PIEZO: now also U3.29 (*GPIO5)
- net PIEZO_GATE: now also R34.1
- net RTS_BASE: now also R33.1
- net RXD0: now also U3.30 (U0RXD/GPIO3)
- net SCL: now also U3.34 (GPIO22)
- net SCLK: now also U3.18 (MTMS/GPIO14/ADC2_CH6)
- net SDA: now also U3.35 (GPIO21)
- net STAT: now also U3.24 (GPIO4/ADC2_CH0)
- net TXD0: now also U3.31 (U0TXD/GPIO1)
- no-connect marks 17 -> 18
Other:
- note added: "MANUAL ENABLE (reset button)"
- note added: "TODO:"
- note added: "chip datasheet claims to not have GPIO34 and GPIO35, but the module datasheet says it does. 34 to 39 are GPI (no output) only and have no builtin pull-ups. GPIO2 and GPIO12 are strapping."
- note added: "test points for voltages, both sides of each diode, BOOT"
- note removed: "10k, 1uf ideally"
- note removed: "MANUAL EN & BOOT"
- note removed: "TODO: BOOT seems to be low on power-up :( probably without cp2102n"
- note removed: "TODO: test points for voltages, both sides of each diode"
- note removed: "finicky as hell"
- moved on the sheet: BZ1, C13, C14, C15, C16, C17, Q1A, Q1B, Q3B, R10, R11, R13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

Commit message: pcb changes
Parts:
- R16, R20, R3, R32, R33, R34: value 100k -> 1M
Other:
- note added: "don't put a pull-down on the piezo pin as it is a strapping pin"
Changed lines of the file:
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@@
+    (effects (font (size 1.27 1.27)) (justify left bottom))
+  )
+  (text "don't put a pull-down on the piezo pin as it is a strapping pin"
+    (at 151.13 66.04 0)
     (effects (font (size 1.27 1.27)) (justify left bottom))
   )
@@
     (in_bom yes) (on_board yes)
     (property "Reference" "R16" (id 0) (at 143.002 26.67 0))
-    (property "Value" "100k" (id 1) (at 143.637 28.702 0))
+    (property "Value" "1M" (id 1) (at 143.637 28.702 0))
     (property "Footprint" "Resistor_SMD:R_0402_1005Metric" (id 2) (at 140.335 27.94 0)
       (effects (font (size 1.27 1.27)) hide)
@@
     (in_bom yes) (on_board yes)
     (property "Reference" "R33" (id 0) (at 109.982 80.645 0))
-    (property "Value" "100k" (id 1) (at 110.617 82.677 0))
+    (property "Value" "1M" (id 1) (at 110.617 82.677 0))
     (property "Footprint" "Resistor_SMD:R_0402_1005Metric" (id 2) (at 107.315 81.915 0)
       (effects (font (size 1.27 1.27)) hide)
@@
     (in_bom yes) (on_board yes)
     (property "Reference" "R20" (id 0) (at 114.935 177.8 90))
-    (property "Value" "100k" (id 1) (at 114.935 181.61 90))
+    (property "Value" "1M" (id 1) (at 114.935 181.61 90))
     (property "Footprint" "Resistor_SMD:R_0402_1005Metric" (id 2) (at 114.935 179.705 0)
       (effects (font (size 1.27 1.27)) hide)
@@
     (in_bom yes) (on_board yes)
     (property "Reference" "R34" (id 0) (at 260.477 66.04 0))
-    (property "Value" "100k" (id 1) (at 261.112 68.072 0))
+    (property "Value" "1M" (id 1) (at 261.112 68.072 0))
     (property "Footprint" "Resistor_SMD:R_0402_1005Metric" (id 2) (at 257.81 67.31 0)
       (effects (font (size 1.27 1.27)) hide)
@@
     (in_bom yes) (on_board yes)
     (property "Reference" "R32" (id 0) (at 109.982 63.5 0))
-    (property "Value" "100k" (id 1) (at 110.617 65.532 0))
+    (property "Value" "1M" (id 1) (at 110.617 65.532 0))
     (property "Footprint" "Resistor_SMD:R_0402_1005Metric" (id 2) (at 107.315 64.77 0)
       (effects (font (size 1.27 1.27)) hide)
@@
     (in_bom yes) (on_board yes)
     (property "Reference" "R3" (id 0) (at 201.295 26.67 0))
-    (property "Value" "100k" (id 1) (at 202.438 28.956 0))
+    (property "Value" "1M" (id 1) (at 202.438 28.956 0))
     (property "Footprint" "Resistor_SMD:R_0402_1005Metric" (id 2) (at 198.755 27.813 0)
       (effects (font (size 1.27 1.27)) hide)
@@
     )
     (path "/d4ed82c4-96b4-4775-957e-6511f8ba6e2e"
-      (reference "R3") (unit 1) (value "100k") (footprint "Resistor_SMD:R_0402_1005Metric")
+      (reference "R3") (unit 1) (value "1M") (footprint "Resistor_SMD:R_0402_1005Metric")
     )
     (path "/48972a92-f8c8-4934-b852-69581122404d"
@@
     )
     (path "/0a20248d-8ffb-4a43-81cc-a4aa3d3bc6f0"
-      (reference "R16") (unit 1) (value "100k") (footprint "Resistor_SMD:R_0402_1005Metric")
+      (reference "R16") (unit 1) (value "1M") (footprint "Resistor_SMD:R_0402_1005Metric")
     )
     (path "/db240f8d-94fe-4d99-8cee-f769c3ab6dec"
@@
     )
     (path "/a11e9c46-579f-4385-9ee6-36980dd27d46"
-      (reference "R20") (unit 1) (value "100k") (footprint "Resistor_SMD:R_0402_1005Metric")
+      (reference "R20") (unit 1) (value "1M") (footprint "Resistor_SMD:R_0402_1005Metric")
     )
     (path "/fb00f92b-bd12-46ef-bc6f-2025fec1e85a"
@@
     )
     (path "/c7c20aa2-e9ec-4f68-9127-dc5ef7a6baff"
-      (reference "R32") (unit 1) (value "100k") (footprint "Resistor_SMD:R_0402_1005Metric")
+      (reference "R32") (unit 1) (value "1M") (footprint "Resistor_SMD:R_0402_1005Metric")
     )
     (path "/58fcfa02-178c-47e4-b188-30e0f1a28842"
-      (reference "R33") (unit 1) (value "100k") (footprint "Resistor_SMD:R_0402_1005Metric")
+      (reference "R33") (unit 1) (value "1M") (footprint "Resistor_SMD:R_0402_1005Metric")
     )
     (path "/b48424f7-b2c0-4591-9463-3edc49682ffd"
-      (reference "R34") (unit 1) (value "100k") (footprint "Resistor_SMD:R_0402_1005Metric")
+      (reference "R34") (unit 1) (value "1M") (footprint "Resistor_SMD:R_0402_1005Metric")
     )
     (path "/4caf1c03-a213-489a-a665-c3f72b156de1"

Commit message: wip
Parts:
- R16, R20: value 1M -> 10k
- R3, R32, R33, R34: value 1M -> 100k
Other:
- note added: "100k???"
- note added: "TODO: remove this, but try and put a low pass filter on the piezo and if that works reuse the same spot on the solder stencil."
- note added: "move the piezo off gpio5. If it is on to a strapping pin, make it one that can be pulled down at boot"
- note added: "use DAC1 & DAC2 rather"
- note removed: "chip datasheet claims to not have GPIO34 and GPIO35, but the module datasheet says it does. 34 to 39 are GPI (no output) only and have no builtin pull-ups. GPIO2 and GPIO12 are strapping."
Changed lines of the file:
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@@
+    (effects (font (size 1.27 1.27)) (justify left bottom))
+  )
+  (text "use DAC1 & DAC2 rather" (at 150.495 64.77 0)
     (effects (font (size 1.27 1.27)) (justify left bottom))
   )
@@
   )
   (text "(ROTARY ENCODER & LCD)" (at 182.245 21.59 0)
+    (effects (font (size 1.27 1.27)) (justify left bottom))
+  )
+  (text "move the piezo off gpio5. If it is on to a strapping pin,\nmake it one that can be pulled down at boot"
+    (at 150.495 61.595 0)
     (effects (font (size 1.27 1.27)) (justify left bottom))
   )
@@
     (effects (font (size 1.27 1.27)) (justify left bottom))
   )
+  (text "100k???" (at 97.155 85.09 0)
+    (effects (font (size 1.27 1.27)) (justify left bottom))
+  )
   (text "USB TO SERIAL" (at 15.494 46.609 0)
     (effects (font (size 1.27 1.27)) (justify left bottom))
   )
+  (text "TODO: remove this, but try and put a\nlow pass filter on the piezo and if\nthat works reuse the same spot on\nthe solder stencil.\n"
+    (at 220.345 72.39 0)
+    (effects (font (size 1.27 1.27)) (justify left bottom))
+  )
   (text "LCD CONNECTOR" (at 79.375 143.891 0)
     (effects (font (size 1.27 1.27)) (justify left bottom))
@@
   )
   (text "don't put a pull-down on the piezo pin as it is a strapping pin"
-    (at 151.13 66.04 0)
+    (at 150.495 57.15 0)
     (effects (font (size 1.27 1.27)) (justify left bottom))
   )
   (text "USB PORT" (at 15.24 17.145 0)
+    (effects (font (size 1.27 1.27)) (justify left bottom))
+  )
+  (text "100k???" (at 96.52 67.31 0)
     (effects (font (size 1.27 1.27)) (justify left bottom))
   )
@@
   )
   (text "Diode because CP2102N is\n5.25V, USB 2 is 5.5V" (at 15.367 51.689 0)
-    (effects (font (size 1.27 1.27)) (justify left bottom))
-  )
-  (text "chip datasheet claims to not have GPIO34 and GPIO35,\nbut the module datasheet says it does.\n34 to 39 are GPI (no output) only and have no builtin pull-ups.\nGPIO2 and GPIO12 are strapping. "
-    (at 150.495 62.23 0)
     (effects (font (size 1.27 1.27)) (justify left bottom))
   )
@@
     (in_bom yes) (on_board yes)
     (property "Reference" "R16" (id 0) (at 143.002 26.67 0))
-    (property "Value" "1M" (id 1) (at 143.637 28.702 0))
+    (property "Value" "10k" (id 1) (at 143.637 28.702 0))
     (property "Footprint" "Resistor_SMD:R_0402_1005Metric" (id 2) (at 140.335 27.94 0)
       (effects (font (size 1.27 1.27)) hide)
@@
     (in_bom yes) (on_board yes)
     (property "Reference" "R33" (id 0) (at 109.982 80.645 0))
-    (property "Value" "1M" (id 1) (at 110.617 82.677 0))
+    (property "Value" "100k" (id 1) (at 110.617 82.677 0))
     (property "Footprint" "Resistor_SMD:R_0402_1005Metric" (id 2) (at 107.315 81.915 0)
       (effects (font (size 1.27 1.27)) hide)
@@
     (in_bom yes) (on_board yes)
     (property "Reference" "R20" (id 0) (at 114.935 177.8 90))
-    (property "Value" "1M" (id 1) (at 114.935 181.61 90))
+    (property "Value" "10k" (id 1) (at 114.935 181.61 90))
     (property "Footprint" "Resistor_SMD:R_0402_1005Metric" (id 2) (at 114.935 179.705 0)
       (effects (font (size 1.27 1.27)) hide)
@@
     (in_bom yes) (on_board yes)
     (property "Reference" "R34" (id 0) (at 260.477 66.04 0))
-    (property "Value" "1M" (id 1) (at 261.112 68.072 0))
+    (property "Value" "100k" (id 1) (at 261.112 68.072 0))
     (property "Footprint" "Resistor_SMD:R_0402_1005Metric" (id 2) (at 257.81 67.31 0)
       (effects (font (size 1.27 1.27)) hide)
@@
     (in_bom yes) (on_board yes)
     (property "Reference" "R32" (id 0) (at 109.982 63.5 0))
-    (property "Value" "1M" (id 1) (at 110.617 65.532 0))
+    (property "Value" "100k" (id 1) (at 110.617 65.532 0))
     (property "Footprint" "Resistor_SMD:R_0402_1005Metric" (id 2) (at 107.315 64.77 0)
       (effects (font (size 1.27 1.27)) hide)
@@
     (in_bom yes) (on_board yes)
     (property "Reference" "R3" (id 0) (at 201.295 26.67 0))
-    (property "Value" "1M" (id 1) (at 202.438 28.956 0))
+    (property "Value" "100k" (id 1) (at 202.438 28.956 0))
     (property "Footprint" "Resistor_SMD:R_0402_1005Metric" (id 2) (at 198.755 27.813 0)
       (effects (font (size 1.27 1.27)) hide)
@@
     )
     (path "/d4ed82c4-96b4-4775-957e-6511f8ba6e2e"
-      (reference "R3") (unit 1) (value "1M") (footprint "Resistor_SMD:R_0402_1005Metric")
+      (reference "R3") (unit 1) (value "100k") (footprint "Resistor_SMD:R_0402_1005Metric")
     )
     (path "/48972a92-f8c8-4934-b852-69581122404d"
@@
     )
     (path "/0a20248d-8ffb-4a43-81cc-a4aa3d3bc6f0"
-      (reference "R16") (unit 1) (value "1M") (footprint "Resistor_SMD:R_0402_1005Metric")
+      (reference "R16") (unit 1) (value "10k") (footprint "Resistor_SMD:R_0402_1005Metric")
     )
     (path "/db240f8d-94fe-4d99-8cee-f769c3ab6dec"
@@
     )
     (path "/a11e9c46-579f-4385-9ee6-36980dd27d46"
-      (reference "R20") (unit 1) (value "1M") (footprint "Resistor_SMD:R_0402_1005Metric")
+      (reference "R20") (unit 1) (value "10k") (footprint "Resistor_SMD:R_0402_1005Metric")
     )
     (path "/fb00f92b-bd12-46ef-bc6f-2025fec1e85a"
@@
     )
     (path "/c7c20aa2-e9ec-4f68-9127-dc5ef7a6baff"
-      (reference "R32") (unit 1) (value "1M") (footprint "Resistor_SMD:R_0402_1005Metric")
+      (reference "R32") (unit 1) (value "100k") (footprint "Resistor_SMD:R_0402_1005Metric")
     )
     (path "/58fcfa02-178c-47e4-b188-30e0f1a28842"
-      (reference "R33") (unit 1) (value "1M") (footprint "Resistor_SMD:R_0402_1005Metric")
+      (reference "R33") (unit 1) (value "100k") (footprint "Resistor_SMD:R_0402_1005Metric")
     )
     (path "/b48424f7-b2c0-4591-9463-3edc49682ffd"
-      (reference "R34") (unit 1) (value "1M") (footprint "Resistor_SMD:R_0402_1005Metric")
+      (reference "R34") (unit 1) (value "100k") (footprint "Resistor_SMD:R_0402_1005Metric")
     )
     (path "/4caf1c03-a213-489a-a665-c3f72b156de1"
